Commit message: 为 LINK_TCP 使用简单几何体，新增简化与仿真用 URDF
- wust_seven_axis_arm.urdf / wust_seven_axis_arm_mujoco.urdf：LINK_TCP 的
  visual 与 collision 由缺失的 meshes/LINK_TCP.STL 改为 0.05m 立方体，
  与 wust_seven_axis_arm_simple.urdf 中的表示保持一致
- 新增 wust_seven_axis_arm_simple.urdf（全连杆简化）、
  wust_seven_axis_arm_mujoco.urdf、wust_seven_axis_arm.xml、wust_rm.xml
- .gitignore 忽略 .vscode/ 与本地试验用的大网格 LINK3.obj

Co-Authored-By: Claude Code <noreply@anthropic.com>

File: modules/arm_planning/wust_seven_axis_arm_description/urdf/wust_seven_axis_arm.urdf (robot description, URDF)
Before this commit: robot wust_seven_axis_arm_description, 11 links, 10 joints
Links:
- link LINK_TCP: geometry collision box size=0.05 0.05 0.05; visual box size=0.05 0.05 0.05
