Commit message: 解决时钟串台问题，去掉视觉引导部分

File: modules/arm_planning/description/wust_heavy_lift_description/urdf/robot.urdf (robot description, URDF)
Before this commit: robot robot, 8 links, 7 joints
Links:
- added link LINK_TCP, mass 0.1; collision mesh filename=package://wust_heavy_lift_description/meshes/LINK_TCP.stl; visual mesh filename=package://wust_heavy_lift_description/meshes/LINK_TCP.stl
- added link camera_link, mass 0.1; collision mesh filename=package://wust_heavy_lift_description/meshes/camera_link.stl; visual mesh filename=package://wust_heavy_lift_description/meshes/camera_link.stl
- added link camera_optical_frame
- link base: geometry collision mesh filename=package://wust_heavy_lift_description/meshes/base_collision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; visual mesh filename=package://wust_heavy_lift_description/meshes/base_collision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
- link link1: geometry collision mesh filename=package://wust_heavy_lift_description/meshes/link1_collisio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; visual mesh filename=package://wust_heavy_lift_description/meshes/link1_collisio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
- link link2: geometry collision mesh filename=package://wust_heavy_lift_description/meshes/link2_collisio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; visual mesh filename=package://wust_heavy_lift_description/meshes/link2_collisio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
- link link3: geometry collision mesh filename=package://wust_heavy_lift_description/meshes/link3_collisio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; visual mesh filename=package://wust_heavy_lift_description/meshes/link3_collisio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
- link link4: geometry collision mesh filename=package://wust_heavy_lift_description/meshes/link4_collisio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; visual mesh filename=package://wust_heavy_lift_description/meshes/link4_collisio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
- link link5: geometry collision mesh filename=package://wust_heavy_lift_description/meshes/link5_collisio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; visual mesh filename=package://wust_heavy_lift_description/meshes/link5_collisio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
- link link6: geometry collision mesh filename=package://wust_heavy_lift_description/meshes/link6_collisio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; visual mesh filename=package://wust_heavy_lift_description/meshes/link6_collisio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
- link link7: geometry collision mesh filename=package://wust_heavy_lift_description/meshes/link7_collisio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; visual mesh filename=package://wust_heavy_lift_description/meshes/link7_collisio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
Joints:
- added joint camera_joint: type fixed, parent link7, child camera_link, origin xyz=0 -0.08 0.04 rpy=3.1416 0 3.1416
- added joint camera_optical_joint: type fixed, parent camera_link, child camera_optical_frame, origin xyz=0 0 0 rpy=0 0 0
- added joint vacuum_tcp: type fixed, parent link7, child LINK_TCP, origin xyz=0.0366 0 -0.081603 rpy=3.1416 0 3.1416
